File: esp8266-dev-board.brd (EAGLE design)
At the start: 25.5 x 33 mm, 9 parts, among them J1 left, J2 right

Commit message: MicroSD shield compatibility
Connections:
- net N$1: now also J1.3; no longer J2.5
- net N$2: now also J2.6; no longer J2.4
- net N$3: now also J2.2; no longer J2.3
Routing:
- net N$1: track 18.4 -> 45.6 mm
- net N$2: track 23.4 -> 18.8 mm
- net N$3: track 20.7 -> 24.5 mm
Changed lines of the file:
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@@
 <grid distance="1" unitdist="mil" unit="mil" style="lines" multiple="1" display="yes" altdistance="0.025" altunitdist="inch" altunit="mm"/>
 <layers>
-<layer number="1" name="Top" color="4" fill="1" visible="no" active="yes"/>
+<layer number="1" name="Top" color="4" fill="1" visible="yes" active="yes"/>
 <layer number="2" name="Route2" color="1" fill="3" visible="no" active="no"/>
 <layer number="3" name="Route3" color="4" fill="3" visible="no" active="no"/>
@@
 <layer number="14" name="Route14" color="1" fill="6" visible="no" active="no"/>
 <layer number="15" name="Route15" color="4" fill="6" visible="no" active="no"/>
-<layer number="16" name="Bottom" color="1" fill="1" visible="no" active="yes"/>
-<layer number="17" name="Pads" color="2" fill="1" visible="no" active="yes"/>
-<layer number="18" name="Vias" color="2" fill="1" visible="no" active="yes"/>
-<layer number="19" name="Unrouted" color="6" fill="1" visible="no" active="yes"/>
-<layer number="20" name="Dimension" color="15" fill="1" visible="no" active="yes"/>
-<layer number="21" name="tPlace" color="7" fill="1" visible="no" active="yes"/>
+<layer number="16" name="Bottom" color="1" fill="1" visible="yes" active="yes"/>
+<layer number="17" name="Pads" color="2" fill="1" visible="yes" active="yes"/>
+<layer number="18" name="Vias" color="2" fill="1" visible="yes" active="yes"/>
+<layer number="19" name="Unrouted" color="6" fill="1" visible="yes" active="yes"/>
+<layer number="20" name="Dimension" color="15" fill="1" visible="yes" active="yes"/>
+<layer number="21" name="tPlace" color="7" fill="1" visible="yes" active="yes"/>
 <layer number="22" name="bPlace" color="7" fill="1" visible="yes" active="yes"/>
-<layer number="23" name="tOrigins" color="15" fill="1" visible="no" active="yes"/>
+<layer number="23" name="tOrigins" color="15" fill="1" visible="yes" active="yes"/>
 <layer number="24" name="bOrigins" color="15" fill="1" visible="yes" active="yes"/>
-<layer number="25" name="tNames" color="7" fill="1" visible="no" active="yes"/>
-<layer number="26" name="bNames" color="7" fill="1" visible="no" active="yes"/>
-<layer number="27" name="tValues" color="7" fill="1" visible="no" active="yes"/>
-<layer number="28" name="bValues" color="7" fill="1" visible="no" active="yes"/>
+<layer number="25" name="tNames" color="7" fill="1" visible="yes" active="yes"/>
+<layer number="26" name="bNames" color="7" fill="1" visible="yes" active="yes"/>
+<layer number="27" name="tValues" color="7" fill="1" visible="yes" active="yes"/>
+<layer number="28" name="bValues" color="7" fill="1" visible="yes" active="yes"/>
 <layer number="29" name="tStop" color="7" fill="3" visible="no" active="yes"/>
 <layer number="30" name="bStop" color="7" fill="6" visible="no" active="yes"/>
@@
 <layer number="37" name="tTest" color="7" fill="1" visible="no" active="yes"/>
 <layer number="38" name="bTest" color="7" fill="1" visible="no" active="yes"/>
-<layer number="39" name="tKeepout" color="4" fill="11" visible="no" active="yes"/>
-<layer number="40" name="bKeepout" color="1" fill="11" visible="no" active="yes"/>
-<layer number="41" name="tRestrict" color="4" fill="10" visible="no" active="yes"/>
-<layer number="42" name="bRestrict" color="1" fill="10" visible="no" active="yes"/>
+<layer number="39" name="tKeepout" color="4" fill="11" visible="yes" active="yes"/>
+<layer number="40" name="bKeepout" color="1" fill="11" visible="yes" active="yes"/>
+<layer number="41" name="tRestrict" color="4" fill="10" visible="yes" active="yes"/>
+<layer number="42" name="bRestrict" color="1" fill="10" visible="yes" active="yes"/>
 <layer number="43" name="vRestrict" color="2" fill="10" visible="no" active="yes"/>
-<layer number="44" name="Drills" color="7" fill="1" visible="no" active="yes"/>
-<layer number="45" name="Holes" color="7" fill="1" visible="no" active="yes"/>
+<layer number="44" name="Drills" color="7" fill="1" visible="yes" active="yes"/>
+<layer number="45" name="Holes" color="7" fill="1" visible="yes" active="yes"/>
 <layer number="46" name="Milling" color="3" fill="1" visible="no" active="yes"/>
 <layer number="47" name="Measures" color="7" fill="1" visible="no" active="yes"/>
@@
 <layer number="49" name="Reference" color="7" fill="1" visible="no" active="yes"/>
 <layer number="50" name="dxf" color="7" fill="1" visible="no" active="no"/>
-<layer number="51" name="tDocu" color="7" fill="1" visible="no" active="yes"/>
-<layer number="52" name="bDocu" color="7" fill="1" visible="no" active="yes"/>
+<layer number="51" name="tDocu" color="7" fill="1" visible="yes" active="yes"/>
+<layer number="52" name="bDocu" color="7" fill="1" visible="yes" active="yes"/>
 <layer number="53" name="tGND_GNDA" color="7" fill="9" visible="no" active="no"/>
 <layer number="54" name="bGND_GNDA" color="1" fill="9" visible="no" active="no"/>
@@
 <layer number="196" name="aValue" color="7" fill="1" visible="no" active="yes"/>
 <layer number="199" name="Contour" color="7" fill="1" visible="no" active="yes"/>
-<layer number="200" name="200bmp" color="1" fill="10" visible="yes" active="yes"/>
+<layer number="200" name="200bmp" color="1" fill="10" visible="no" active="yes"/>
 <layer number="201" name="201bmp" color="2" fill="1" visible="no" active="no"/>
 <layer number="202" name="202bmp" color="3" fill="1" visible="no" active="no"/>
@@
 <contactref element="C1" pad="2"/>
 </signal>
-<signal name="N$1">
-<contactref element="J2" pad="5"/>
-<contactref element="U$1" pad="5"/>
-<wire x1="9.43" y1="24.13" x2="9.43" y2="23.59" width="0.4064" layer="1"/>
-<wire x1="9.43" y1="23.59" x2="11.43" y2="21.59" width="0.4064" layer="1"/>
-<wire x1="11.43" y1="21.59" x2="17.78" y2="21.59" width="0.4064" layer="1"/>
-<wire x1="17.78" y1="21.59" x2="19.05" y2="20.32" width="0.4064" layer="1"/>
-<wire x1="19.05" y1="20.32" x2="19.05" y2="17.78" width="0.4064" layer="1"/>
-<wire x1="19.05" y1="17.78" x2="20.32" y2="16.51" width="0.4064" layer="1"/>
-<wire x1="20.32" y1="16.51" x2="22.86" y2="16.51" width="0.4064" layer="1"/>
-</signal>
 <signal name="D1">
 <contactref element="J1" pad="6"/>
@@
 <signal name="N$2">
 <contactref element="U$1" pad="2"/>
-<contactref element="J2" pad="4"/>
-<wire x1="22.86" y1="13.97" x2="21.59" y2="13.97" width="0.4064" layer="16"/>
-<wire x1="21.59" y1="13.97" x2="20.32" y2="15.24" width="0.4064" layer="16"/>
-<wire x1="20.32" y1="15.24" x2="20.32" y2="26.67" width="0.4064" layer="16"/>
-<wire x1="20.32" y1="26.67" x2="19.05" y2="27.94" width="0.4064" layer="16"/>
+<wire x1="19.05" y1="27.94" x2="20.32" y2="26.67" width="0.4064" layer="16"/>
 <wire x1="19.05" y1="27.94" x2="13.97" y2="27.94" width="0.4064" layer="16"/>
 <wire x1="13.43" y1="26.13" x2="13.43" y2="27.4" width="0.4064" layer="16"/>
 <wire x1="13.43" y1="27.4" x2="13.97" y2="27.94" width="0.4064" layer="16"/>
+<contactref element="J2" pad="6"/>
+<wire x1="20.32" y1="26.67" x2="20.32" y2="19.5834" width="0.4064" layer="16"/>
+<wire x1="20.32" y1="19.5834" x2="20.8788" y2="19.0246" width="0.4064" layer="16"/>
+<wire x1="20.8788" y1="19.0246" x2="22.8346" y2="19.0246" width="0.4064" layer="16"/>
+<wire x1="22.8346" y1="19.0246" x2="22.86" y2="19.05" width="0.4064" layer="16"/>
 </signal>
 <signal name="N$3">
-<contactref element="J2" pad="3"/>
 <contactref element="U$1" pad="3"/>
 <wire x1="11.43" y1="24.13" x2="12.7" y2="22.86" width="0.4064" layer="16"/>
 <wire x1="12.7" y1="22.86" x2="17.78" y2="22.86" width="0.4064" layer="16"/>
-<wire x1="22.86" y1="11.43" x2="22.67" y2="11.62" width="0.4064" layer="16"/>
-<wire x1="22.67" y1="11.62" x2="22.19" y2="11.62" width="0.4064" layer="16"/>
-<wire x1="22.19" y1="11.62" x2="18.85" y2="14.96" width="0.4064" layer="16"/>
-<wire x1="18.85" y1="14.96" x2="18.85" y2="21.79" width="0.4064" layer="16"/>
+<wire x1="18.85" y1="21.79" x2="18.85" y2="14.96" width="0.4064" layer="16"/>
 <wire x1="18.85" y1="21.79" x2="17.78" y2="22.86" width="0.4064" layer="16"/>
+<contactref element="J2" pad="2"/>
+<wire x1="18.85" y1="14.96" x2="20.2946" y2="13.5154" width="0.4064" layer="16"/>
+<wire x1="20.2946" y1="13.5154" x2="20.2946" y2="8.8646" width="0.4064" layer="16"/>
+<wire x1="20.2946" y1="8.8646" x2="22.8346" y2="8.8646" width="0.4064" layer="16"/>
+<wire x1="22.8346" y1="8.8646" x2="22.86" y2="8.89" width="0.1524" layer="16"/>
 </signal>
 <signal name="D2">
@@
 <wire x1="12.18201875" y1="1.27" x2="13.14701875" y2="2.235" width="0.4064" layer="1"/>
 </signal>
+<signal name="N$1">
+<contactref element="J1" pad="3"/>
+<contactref element="U$1" pad="5"/>
+<wire x1="10.9656" y1="9.82630625" x2="10.9474" y2="9.80810625" width="0.4064" layer="16"/>
+<wire x1="10.9474" y1="9.80810625" x2="10.9474" y2="-0.0254" width="0.4064" layer="16"/>
+<wire x1="9.43" y1="24.13" x2="10.9656" y2="22.5944" width="0.4064" layer="16"/>
+<wire x1="10.9656" y1="22.5944" x2="10.9656" y2="9.82630625" width="0.4064" layer="16"/>
+<wire x1="10.9474" y1="-0.0254" x2="3.1242" y2="-0.0254" width="0.4064" layer="16"/>
+<wire x1="1.4986" y1="1.6002" x2="1.4986" y2="10.3886" width="0.4064" layer="16"/>
+<wire x1="1.4986" y1="10.3886" x2="0.4572" y2="11.43" width="0.4064" layer="16"/>
+<wire x1="0.4572" y1="11.43" x2="0" y2="11.43" width="0.4064" layer="16"/>
+<wire x1="3.1242" y1="-0.0254" x2="1.4986" y2="1.6002" width="0.4064" layer="16"/>
+</signal>
 </signals>
